File: KiCAD/ERK01_PSU/ERK01_PSU.kicad_pcb (KiCad board)
At the start: 2 copper layers, 71.1 x 45.7 mm, 24 parts, among them J1 PWR_IN, J2 TP_GND, J3 PWR_OUT_1, J4 PWR_OUT_2, U1 L7812, U2 L7912

Commit message: Add: Panel Size
Parts:
- added H5: MountingHole, MountingHole:MountingHole_2.2mm_M2, F.Cu at (119.4, 81.3)
- added H6: MountingHole, MountingHole:MountingHole_2.2mm_M2, F.Cu at (119.4, 116.8)
Routing:
- net /+5V: track 100.7 -> 102.8 mm
Changed lines of the file:
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@@
     (thickness 1.6)
     (drawings 378)
-    (tracks 115)
+    (tracks 117)
     (zones 0)
-    (modules 24)
+    (modules 26)
     (nets 11)
   )
@@
     (add_net "Net-(D6-Pad1)")
   )
+  (module MountingHole:MountingHole_2.2mm_M2 (layer F.Cu)
+    (at 119.38 116.84)
+    (descr "Mounting Hole 2.2mm, no annular, M2")
+    (tags "mounting hole 2.2mm no annular m2")
+    (attr virtual)
+    (fp_text reference H6 (at -3.72 0.15) (layer F.SilkS)
+      (effects (font (size 1 1) (thickness 0.15)))
+    )
+    (fp_text value MountingHole (at 0 3.2) (layer F.Fab)
+      (effects (font (size 1 1) (thickness 0.15)))
+    )
+    (fp_circle (center 0 0) (end 2.45 0) (layer F.CrtYd) (width 0.05))
+    (fp_circle (center 0 0) (end 2.2 0) (layer Cmts.User) (width 0.15))
+    (fp_text user %R (at 0.3 0) (layer F.Fab)
+      (effects (font (size 1 1) (thickness 0.15)))
+    )
+    (pad 1 np_thru_hole circle (at 0 0) (size 2.2 2.2) (drill 2.2) (layers *.Cu *.Mask))
+  )
+  (module MountingHole:MountingHole_2.2mm_M2 (layer F.Cu)
+    (at 119.38 81.28)
+    (descr "Mounting Hole 2.2mm, no annular, M2")
+    (tags "mounting hole 2.2mm no annular m2")
+    (attr virtual)
+    (fp_text reference H5 (at -3.96 -0.55) (layer F.SilkS)
+      (effects (font (size 1 1) (thickness 0.15)))
+    )
+    (fp_text value MountingHole (at 7.62 -1.27) (layer F.Fab)
+      (effects (font (size 1 1) (thickness 0.15)))
+    )
+    (fp_circle (center 0 0) (end 2.45 0) (layer F.CrtYd) (width 0.05))
+    (fp_circle (center 0 0) (end 2.2 0) (layer Cmts.User) (width 0.15))
+    (fp_text user %R (at 0.3 0) (layer F.Fab)
+      (effects (font (size 1 1) (thickness 0.15)))
+    )
+    (pad 1 np_thru_hole circle (at 0 0) (size 2.2 2.2) (drill 2.2) (layers *.Cu *.Mask))
+  )
   (module Capacitor_THT:C_Disc_D3.0mm_W1.6mm_P2.50mm (layer F.Cu)
     (at 121.92 109.22 180)
     (descr "C, Disc series, Radial, pin pitch=2.50mm, , diameter*width=3.0*1.6mm^2, Capacitor, http://www.vishay.com/docs/45233/krseries.pdf")
     (tags "C Disc series Radial pin pitch 2.50mm  diameter 3.0mm width 1.6mm Capacitor")
-    (fp_text reference C2 (at 1.25 -2.05) (layer F.SilkS)
-      (effects (font (size 1 1) (thickness 0.15)))
-    )
-    (fp_text value 0.33uF (at 1.25 2.05) (layer F.Fab)
+    (fp_text reference C2 (at -2.59 0.06) (layer F.SilkS)
+      (effects (font (size 1 1) (thickness 0.15)))
+    )
+    (fp_text value 0.33uF (at -3.69 0.09) (layer F.Fab)
       (effects (font (size 1 1) (thickness 0.15)))
     )
@@
     (descr "C, Disc series, Radial, pin pitch=2.50mm, , diameter*width=3.0*1.6mm^2, Capacitor, http://www.vishay.com/docs/45233/krseries.pdf")
     (tags "C Disc series Radial pin pitch 2.50mm  diameter 3.0mm width 1.6mm Capacitor")
-    (fp_text reference C1 (at 1.25 -2.05) (layer F.SilkS)
-      (effects (font (size 1 1) (thickness 0.15)))
-    )
-    (fp_text value 0.33uF (at 1.25 2.05) (layer F.Fab)
+    (fp_text reference C1 (at 5.08 1.27) (layer F.SilkS)
+      (effects (font (size 1 1) (thickness 0.15)))
+    )
+    (fp_text value 0.33uF (at 6.35 0) (layer F.Fab)
       (effects (font (size 1 1) (thickness 0.15)))
     )
@@
       (effects (font (size 1 1) (thickness 0.15)))
     )
-    (fp_text value 1S4 (at 3.81 1.92) (layer F.Fab)
+    (fp_text value 1S4 (at 6.46 -1.97) (layer F.Fab)
       (effects (font (size 1 1) (thickness 0.15)))
     )
@@
     (descr "Diode, DO-34_SOD68 series, Axial, Horizontal, pin pitch=7.62mm, , length*diameter=3.04*1.6mm^2, , https://www.nxp.com/docs/en/data-sheet/KTY83_SER.pdf")
     (tags "Diode DO-34_SOD68 series Axial Horizontal pin pitch 7.62mm  length 3.04mm diameter 1.6mm")
-    (fp_text reference D1 (at 3.81 -1.92) (layer F.SilkS)
+    (fp_text reference D1 (at 6.604 2.032) (layer F.SilkS)
       (effects (font (size 1 1) (thickness 0.15)))
     )
@@
     (descr "TO-220-3, Vertical, RM 2.54mm, see https://www.vishay.com/docs/66542/to-220-1.pdf")
     (tags "TO-220-3 Vertical RM 2.54mm")
-    (fp_text reference U2 (at 2.54 -4.27) (layer F.SilkS)
-      (effects (font (size 1 1) (thickness 0.15)))
-    )
-    (fp_text value L7912 (at 2.54 2.5) (layer F.Fab)
-      (effects (font (size 1 1) (thickness 0.15)))
-    )
-    (fp_text user %R (at 2.54 -4.27) (layer F.Fab)
+    (fp_text reference U2 (at -3.82 -2.84) (layer F.SilkS)
+      (effects (font (size 1 1) (thickness 0.15)))
+    )
+    (fp_text value L7912 (at -2.55 -4.21) (layer F.Fab)
+      (effects (font (size 1 1) (thickness 0.15)))
+    )
+    (fp_text user %R (at -3.84 -1.2) (layer F.Fab)
       (effects (font (size 1 1) (thickness 0.15)))
     )
@@
     (descr "TO-220-3, Vertical, RM 2.54mm, see https://www.vishay.com/docs/66542/to-220-1.pdf")
     (tags "TO-220-3 Vertical RM 2.54mm")
-    (fp_text reference U1 (at 2.54 -4.27) (layer F.SilkS)
-      (effects (font (size 1 1) (thickness 0.15)))
-    )
-    (fp_text value L7812 (at 2.54 2.5) (layer F.Fab)
+    (fp_text reference U1 (at 8.89 -4.064) (layer F.SilkS)
+      (effects (font (size 1 1) (thickness 0.15)))
+    )
+    (fp_text value L7812 (at 10.16 -2.54) (layer F.Fab)
       (effects (font (size 1 1) (thickness 0.15)))
     )
@@
     (descr "Through hole straight pin header, 1x02, 2.54mm pitch, single row")
     (tags "Through hole pin header THT 1x02 2.54mm single row")
-    (fp_text reference J2 (at 0 -2.33) (layer F.SilkS)
+    (fp_text reference J2 (at 3.06 3.11) (layer F.SilkS)
       (effects (font (size 1 1) (thickness 0.15)))
     )
@@
     (descr "JST XH series connector, B5B-XH-A (http://www.jst-mfg.com/product/pdf/eng/eXH.pdf), generated with kicad-footprint-generator")
     (tags "connector JST XH vertical")
-    (fp_text reference J1 (at 5 -3.55 90) (layer F.SilkS)
+    (fp_text reference J1 (at -4.32 3 90) (layer F.SilkS)
       (effects (font (size 1 1) (thickness 0.15)))
     )
@@
       (effects (font (size 1 1) (thickness 0.15)))
     )
-    (fp_text value 470uF (at 2.5 6.25 90) (layer F.Fab)
+    (fp_text value 470uF (at 7.93 4.95 90) (layer F.Fab)
       (effects (font (size 1 1) (thickness 0.15)))
     )
@@
       (effects (font (size 1 1) (thickness 0.15)))
     )
-    (fp_text value 470uF (at 2.5 6.25 90) (layer F.Fab)
+    (fp_text value 470uF (at 7.27 5.19 90) (layer F.Fab)
       (effects (font (size 1 1) (thickness 0.15)))
     )
@@
     (descr "C, Disc series, Radial, pin pitch=2.50mm, , diameter*width=3.0*1.6mm^2, Capacitor, http://www.vishay.com/docs/45233/krseries.pdf")
     (tags "C Disc series Radial pin pitch 2.50mm  diameter 3.0mm width 1.6mm Capacitor")
-    (fp_text reference C4 (at 1.25 -2.05) (layer F.SilkS)
-      (effects (font (size 1 1) (thickness 0.15)))
-    )
-    (fp_text value 0.1uF (at 1.25 2.05) (layer F.Fab)
+    (fp_text reference C4 (at -1.65 1.97) (layer F.SilkS)
+      (effects (font (size 1 1) (thickness 0.15)))
+    )
+    (fp_text value 0.1uF (at -2.27 1.87) (layer F.Fab)
       (effects (font (size 1 1) (thickness 0.15)))
     )
@@
     (descr "C, Disc series, Radial, pin pitch=2.50mm, , diameter*width=3.0*1.6mm^2, Capacitor, http://www.vishay.com/docs/45233/krseries.pdf")
     (tags "C Disc series Radial pin pitch 2.50mm  diameter 3.0mm width 1.6mm Capacitor")
-    (fp_text reference C3 (at 1.25 -2.05) (layer F.SilkS)
-      (effects (font (size 1 1) (thickness 0.15)))
-    )
-    (fp_text value 0.1uF (at 1.25 2.05) (layer F.Fab)
+    (fp_text reference C3 (at -4.67 1.05) (layer F.SilkS)
+      (effects (font (size 1 1) (thickness 0.15)))
+    )
+    (fp_text value 0.1uF (at -5.15 0.66) (layer F.Fab)
       (effects (font (size 1 1) (thickness 0.15)))
     )
@@
     )
   )
-  (gr_text https://dad8893.blogspot.com/ (at 134.62 120.65) (layer F.SilkS)
+  (gr_text https://dad8893.blogspot.com/ (at 139.7 120.65) (layer F.SilkS)
     (effects (font (size 1 1) (thickness 0.2)))
   )
-  (gr_text "ERK01_PSU V.1.0" (at 132.08 118.11) (layer F.SilkS)
+  (gr_text "ERK01_PSU V.1.0" (at 139.7 118.11) (layer F.SilkS)
     (effects (font (size 1.5 1.5) (thickness 0.3)))
   )
@@
   (segment (start 170.18 86.36) (end 170.18 93.98) (width 0.5) (layer B.Cu) (net 8))
   (segment (start 165.1 81.28) (end 170.18 86.36) (width 0.5) (layer B.Cu) (net 8))
-  (segment (start 111.76 81.28) (end 165.1 81.28) (width 0.5) (layer B.Cu) (net 8))
   (segment (start 106.68 93.98) (end 106.68 86.36) (width 0.5) (layer B.Cu) (net 8))
   (segment (start 106.68 86.36) (end 111.76 81.28) (width 0.5) (layer B.Cu) (net 8))
@@
   (segment (start 167.64 93.98) (end 170.18 93.98) (width 0.5) (layer B.Cu) (net 8))
   (segment (start 154.94 93.98) (end 157.48 93.98) (width 0.5) (layer B.Cu) (net 8))
+  (segment (start 111.76 81.28) (end 114.3 78.74) (width 0.5) (layer B.Cu) (net 8))
+  (segment (start 114.3 78.74) (end 162.56 78.74) (width 0.5) (layer B.Cu) (net 8))
+  (segment (start 162.56 78.74) (end 165.1 81.28) (width 0.5) (layer B.Cu) (net 8))
   (segment (start 165.1 91.44) (end 167.64 91.44) (width 0.5) (layer B.Cu) (net 9))
   (segment (start 152.4 91.44) (end 154.94 91.44) (width 0.5) (layer B.Cu) (net 9))
